Commit message: Added inertial property such as mass, inertia to the kheperas. The rviz gives a warning about the base link does not support an inertia value. This need to be deal with if futhure problems come across. Other than this, the inertial properties loaded corrected.

File: kheperas_description/urdf/kheperas_base.urdf (robot description, URDF)
Before this commit: robot kheperas, 5 links, 4 joints
Links:
- link back_caster_link: mass None -> 0.0061
- link base_link: mass None -> 1.06
- link front_caster_link: mass None -> 0.0061
- link left_wheel_link: mass None -> 0.021
- link right_wheel_link: mass None -> 0.021

Commit message: Fixed the wheel rotation axis.

File: kheperas_description/urdf/kheperas_base.urdf (robot description, URDF)
Before this commit: robot kheperas, 5 links, 4 joints
Joints:
- joint left_wheel_joint: axis 0.0 1.0 0.0 -> 0.0 0.0 1.0
- joint right_wheel_joint: axis 0.0 1.0 0.0 -> 0.0 0.0 1.0
