Commit message: i have tried again to use xacro to format the kheperas urdf but it does not work again, i have no idea why. SO i move back to the standard urdf format to code it in the original way. The robot spawn in the gazebo nicely but it has a werid moving which is not desired.

File: kheperas_description/urdf/urdf/kheperas_base_gazebo.urdf (robot description, URDF)
Before this commit: robot kheperas, 6 links, 5 joints
Links:
- link base_link: geometry collision cylinder length=0.053 radius=0.07004; visual cylinder length=0.053 radius=0.07004
- link left_wheel_link: geometry collision cylinder length=0.0059 radius=0.021; visual cylinder length=0.0059 radius=0.021
- link right_wheel_link: geometry collision cylinder length=0.0059 radius=0.021; visual cylinder length=0.0059 radius=0.021

Commit message: there is a controller yaml file made to replace the gazebo hardcoded diff_drive in order to rule out the reason why the robot has a random swift. The problem has finally been pinned to the urdf file which is the geometry of the robot. The swift happens due to there is not enough contact file for the robot to be dynamic stable and it is finally been solved. the gazebo simulation is now stable.

File: kheperas_description/urdf/urdf/kheperas_base_gazebo.urdf (robot description, URDF)
Before this commit: robot kheperas, 6 links, 5 joints
Links:
- link left_wheel_link: geometry collision cylinder length=0.0030 radius=0.015; visual cylinder length=0.0059 radius=0.021
- link right_wheel_link: geometry collision cylinder length=0.0030 radius=0.015; visual cylinder length=0.0059 radius=0.021

File: kheperas_description/urdf/urdf/kheperas_wLaser_gazebo.urdf (robot description, URDF)
Before this commit: robot kheperas, 7 links, 6 joints
Links:
- link back_caster_link: geometry collision sphere radius=0.01134; visual sphere radius=0.01134
- link front_caster_link: geometry collision sphere radius=0.01134; visual sphere radius=0.01134
