Commit message: Added in a imu sensor which linked to the base_link of the Kheperas robot.

File: kheperas_description/urdf/urdf/kheperas_wLaser_gazebo.urdf (robot description, URDF)
Before this commit: robot kheperas, 7 links, 6 joints
Joints:
- joint base_l_wheel_joint: parent base_link -> base_footprint
- joint base_r_wheel_joint: parent base_link -> base_footprint
- joint laser_joint: origin xyz=0.0 0.0 0.053 rpy=0.0 0.0 0.0 -> xyz=0.0 0.0 0.0265 rpy=0.0 0.0 0.0
