Commit message: change the old kheperas_base_gazebo.urdf to --_reference_-- added in a laser and seperate topic published onto the same one into difference topic name

File: kheperas_description/urdf/urdf/kheperas_reference_gazebo.urdf (robot description, URDF)
Before this commit: robot kheperas, 6 links, 5 joints
Links:
- added link laser_link, mass 0.1; collision cylinder length=0.06 radius=0.05; visual cylinder length=0.02 radius=0.02
- link back_caster_link: geometry collision sphere radius=0.01134; visual sphere radius=0.01134
- link front_caster_link: geometry collision sphere radius=0.01134; visual sphere radius=0.01134
- link left_wheel_link: geometry collision cylinder length=0.0059 radius=0.021; visual cylinder length=0.0059 radius=0.021
- link right_wheel_link: geometry collision cylinder length=0.0059 radius=0.021; visual cylinder length=0.0059 radius=0.021
Joints:
- added joint laser_joint: type fixed, parent base_link, child laser_link, origin xyz=0.0 0.0 0.0265 rpy=0.0 0.0 0.0
