Commit message: improve the launch file codes, there are four robots spawning for the purpose of tkf model testing.

File: kheperas_description/urdf/urdf/kheperas.urdf (robot description, URDF)
Before this commit: robot kheperas, 8 links, 7 joints
Joints:
- joint base_l_wheel_joint: parent base_footprint -> base_link
- joint base_r_wheel_joint: parent base_footprint -> base_link

File: kheperas_description/urdf/urdf/kheperas_base_gazebo.urdf (robot description, URDF)
Before this commit: robot kheperas, 7 links, 6 joints
Links:
- removed link laser_link
Joints:
- removed joint laser_joint

Commit message: slight chagne is made

File: kheperas_description/urdf/urdf/kheperas.urdf (robot description, URDF)
Before this commit: robot kheperas, 8 links, 7 joints
Links:
- link camera_link: geometry collision box size=0.02 0.02 0.01; visual box size=0.007 0.02 0.02
